File: NAND_SD.kicad_sch (KiCad schematic)
At the start: 8 parts, among them U10 F35SQA512M-WWT

Commit message: power changes for v3s, cleanup
Other:
- title: (none) -> iPodClone
Changed lines of the file:
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@@
 	(generator_version "9.0")
 	(paper "A4")
+	(title_block
+		(title "iPodClone")
+		(rev "1.0")
+		(comment 1 "microSD for file system and NAND flash for boot")
+	)
 	(text "make sure hold\nshould be pulled\nhigh"
 		(exclude_from_sim no)
