File: WiFiBT.kicad_sch (KiCad schematic)
At the start: 1 part, among them U2 ESP32-D0WD-V3

Commit message: before switching to ESP32 module
Parts:
- added C30, C31, C34, C35: 0.1uF, symbol Device:C
- added C32, C37: 1uF, symbol Device:C
- added C33: 10uF, symbol Device:C
- added C36: 100pF, symbol Device:C
- added C38, C39: C, symbol Device:C
- added L5: 2nH, symbol Device:L
- added X2: XTM32040000JT00351005, easyeda2kicad:CRYSTAL-SMD_4P-L3.2-W2.5-BL, symbol easyeda2kicad:XTM32040000JT00351005
Connections:
- net +3.3V: now reaches U2.1 (VDDA)
- net +3.3V: now also U2.19 (VDD3P3_RTC), U2.37 (VDD3P3_CPU), U2.43 (VDDA), U2.46 (VDDA), C30.1, C31.1, C32.1, C33.1, C34.1, C35.1, C36.1, C37.1, L5.1
- net at U2.3 (VDD3P3): now also U2.4 (VDD3P3), L5.2
- net XTAL_N: now reaches U2.44 (XTAL_N)
- net XTAL_N: now also C38.1, X2.3
- net XTAL_P: now reaches U2.45 (XTAL_P)
- net XTAL_P: now also C39.1, X2.1
- net GND: now reaches U2.49 (GND)
- net GND: now also C30.2, C31.2, C32.2, C33.2, C34.2, C35.2, C36.2, C37.2, C38.2, C39.2, X2.2 (GND), X2.4 (GND)
Other:
- moved on the sheet: U2

Commit message: start of adding esp32 module
Parts:
- removed C34, C35: 0.1uF, symbol Device:C
- removed C36: 100pF, symbol Device:C
- removed C37: 1uF, symbol Device:C
- removed C38, C39: C, symbol Device:C
- removed L5: 2nH, symbol Device:L
- removed U2: ESP32-D0WD-V3, easyeda2kicad:QFN-48_L5.0-W5.0-P0.35-BL-EP3.7, symbol easyeda2kicad:ESP32-D0WD-V3
- removed X2: XTM32040000JT00351005, easyeda2kicad:CRYSTAL-SMD_4P-L3.2-W2.5-BL, symbol easyeda2kicad:XTM32040000JT00351005
- added JP1, JP2: SolderJumper_2_Open, symbol Jumper:SolderJumper_2_Open
- added R25: 10K, symbol Device:R
- added U2: ESP32-MINI-1-H4, easyeda2kicad:WIFI-SMD_ESP32-MINI-1, symbol easyeda2kicad:ESP32-MINI-1-H4
- C33: value 10uF -> 0.1uF
Connections:
- net +3.3V: now also R25.1, U2.3 (3V3); no longer C32.1, C33.1
- net GND: now also JP1.2 (B), JP2.2 (B), U2.1 (GND), U2.2 (GND), U2.27 (GND), U2.38 (GND), U2.39 (GND), U2.40 (GND), U2.41 (GND), U2.42 (GND), U2.43 (GND), U2.44 (GND), U2.45 (GND), U2.46 (GND), U2.47 (GND), U2.48 (GND), U2.49 (GND), U2.50 (GND), U2.51 (GND), U2.52 (GND), U2.53 (GND), U2.54 (GND), U2.55 (GND)
- new net EN: C32.1, C33.1, JP1.1 (A), R25.2, U2.8 (EN)
- new net I2S_MCLK: JP2.1 (A), U2.21 (IO0)
- new net I2S_PCMOUT: U2.29 (IO5)
- new net I2S_SCK: U2.30 (IO18)
- new net I2S_WS: U2.31 (IO23)
- new net RXD0: U2.35 (RXD0)
- new net TCK: U2.18 (IO13)
- new net TDI: U2.17 (IO12)
- new net TDO: U2.19 (IO15)
- new net TMS: U2.16 (IO14)
- new net TXD0: U2.36 (TXD0)
- no-connect marks 0 -> 4
Other:
- note added: "JTAG"
- note added: "Reset jumper for debug"
- note added: "UART0"

Commit message: power changes for v3s, cleanup
Other:
- note added: "I2S Interface"
- title: (none) -> iPodClone
Changed lines of the file:
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@@
 	(generator_version "9.0")
 	(paper "A4")
+	(title_block
+		(title "iPodClone")
+		(rev "1.0")
+		(comment 1 "ESP32 module is used for WiFi and Bluetooth connections")
+	)
 	(rectangle
 		(start 129.286 54.102)
@@
 	)
 	(rectangle
+		(start 20.32 26.67)
+		(end 57.785 50.8)
+		(stroke
+			(width 0)
+			(type dash)
+		)
+		(fill
+			(type none)
+		)
+	)
+	(rectangle
 		(start 224.282 29.464)
 		(end 268.478 59.182)
@@
 		)
 	)
+	(text "I2S Interface"
+		(exclude_from_sim no)
+		(at 26.416 25.4 0)
+		(effects
+			(font
+				(size 1.27 1.27)
+			)
+		)
+	)
 	(text "JTAG\n"
 		(exclude_from_sim no)
@@
 	(wire
 		(pts
-			(xy 55.88 85.09) (xy 48.26 85.09)
+			(xy 46.99 40.64) (xy 39.37 40.64)
 		)
 		(stroke
@@
 	(wire
 		(pts
-			(xy 55.88 80.01) (xy 48.26 80.01)
+			(xy 46.99 35.56) (xy 39.37 35.56)
 		)
 		(stroke
@@
 	(wire
 		(pts
-			(xy 48.26 87.63) (xy 55.88 87.63)
+			(xy 39.37 43.18) (xy 46.99 43.18)
 		)
 		(stroke
@@
 	(wire
 		(pts
-			(xy 55.88 82.55) (xy 48.26 82.55)
+			(xy 46.99 38.1) (xy 39.37 38.1)
 		)
 		(stroke
@@
 	)
 	(label "IO5"
-		(at 55.88 80.01 0)
+		(at 46.99 35.56 0)
 		(effects
 			(font
@@
 	)
 	(label "IO23"
-		(at 55.88 85.09 0)
+		(at 46.99 40.64 0)
 		(effects
 			(font
@@
 	)
 	(label "IO0"
-		(at 55.88 87.63 0)
+		(at 46.99 43.18 0)
 		(effects
 			(font
@@
 	)
 	(label "IO18"
-		(at 55.88 82.55 0)
+		(at 46.99 38.1 0)
 		(effects
 			(font
@@
 	(global_label "I2S_SCK"
 		(shape input)
-		(at 48.26 82.55 180)
+		(at 39.37 38.1 180)
 		(fields_autoplaced yes)
 		(effects
@@
 		)
 		(property "Intersheetrefs" "${INTERSHEET_REFS}"
-			(at 37.5339 82.55 0)
+			(at 28.6439 38.1 0)
 			(effects
 				(font
@@
 	(global_label "I2S_WS"
 		(shape input)
-		(at 48.26 85.09 180)
+		(at 39.37 40.64 180)
 		(fields_autoplaced yes)
 		(effects
@@
 		)
 		(property "Intersheetrefs" "${INTERSHEET_REFS}"
-			(at 38.6225 85.09 0)
+			(at 29.7325 40.64 0)
 			(effects
 				(font
@@
 	(global_label "I2S_PCMOUT"
 		(shape input)
-		(at 48.26 80.01 180)
+		(at 39.37 35.56 180)
 		(fields_autoplaced yes)
 		(effects
@@
 		)
 		(property "Intersheetrefs" "${INTERSHEET_REFS}"
-			(at 33.6634 80.01 0)
+			(at 24.7734 35.56 0)
 			(effects
 				(font
@@
 	(global_label "I2S_MCLK"
 		(shape input)
-		(at 48.26 87.63 180)
+		(at 39.37 43.18 180)
 		(fields_autoplaced yes)
 		(effects
@@
 		)
 		(property "Intersheetrefs" "${INTERSHEET_REFS}"
-			(at 36.2639 87.63 0)
+			(at 27.3739 43.18 0)
 			(effects
 				(font

Commit message: gitignore and audio changes
Connections:
- net V3S-ESP32_TX: now reaches U2.25 (IO9)
- net V3S-ESP32_RX: now reaches U2.26 (IO10)
- net TCK: no longer names the net of U2.18 (IO13)
- net TDI: no longer names the net of U2.17 (IO12)
- net TDO: no longer names the net of U2.19 (IO15)
- net TMS: no longer names the net of U2.16 (IO14)
- no-connect marks 4 -> 24
Other:
- note removed: "JTAG"
Changed lines of the file:
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@@
-	)
-	(rectangle
-		(start 129.286 54.102)
-		(end 141.732 59.182)
-		(stroke
-			(width 0)
-			(type dash)
-		)
-		(fill
-			(type none)
-		)
 	)
 	(rectangle
@@
 		)
 	)
-	(text "JTAG\n"
-		(exclude_from_sim no)
-		(at 131.318 53.086 0)
-		(effects
-			(font
-				(size 1.27 1.27)
-			)
-		)
-	)
 	(text "Reset jumper for debug"
 		(exclude_from_sim no)
@@
 	)
 	(no_connect
+		(at 157.48 83.82)
+	)
+	(no_connect
+		(at 157.48 91.44)
+	)
+	(no_connect
+		(at 101.6 86.36)
+	)
+	(no_connect
+		(at 142.24 63.5)
+	)
+	(no_connect
+		(at 157.48 96.52)
+	)
+	(no_connect
+		(at 157.48 81.28)
+	)
+	(no_connect
 		(at 101.6 76.2)
 	)
 	(no_connect
+		(at 101.6 91.44)
+	)
+	(no_connect
+		(at 132.08 63.5)
+	)
+	(no_connect
+		(at 134.62 63.5)
+	)
+	(no_connect
+		(at 157.48 99.06)
+	)
+	(no_connect
+		(at 157.48 86.36)
+	)
+	(no_connect
 		(at 119.38 63.5)
 	)
 	(no_connect
+		(at 157.48 76.2)
+	)
+	(no_connect
+		(at 124.46 63.5)
+	)
+	(no_connect
+		(at 101.6 88.9)
+	)
+	(no_connect
+		(at 144.78 63.5)
+	)
+	(no_connect
+		(at 157.48 93.98)
+	)
+	(no_connect
+		(at 129.54 63.5)
+	)
+	(no_connect
+		(at 157.48 78.74)
+	)
+	(no_connect
 		(at 101.6 99.06)
 	)
@@
 		(at 121.92 63.5)
 	)
+	(no_connect
+		(at 137.16 63.5)
+	)
+	(no_connect
+		(at 139.7 63.5)
+	)
 	(wire
 		(pts
@@
 	(wire
 		(pts
-			(xy 132.08 58.42) (xy 132.08 63.5)
-		)
-		(stroke
-			(width 0)
-			(type default)
-		)
-	)
-	(wire
-		(pts
 			(xy 93.98 96.52) (xy 101.6 96.52)
 		)
@@
 	(wire
 		(pts
-			(xy 139.7 58.42) (xy 139.7 63.5)
-		)
-		(stroke
-			(width 0)
-			(type default)
-		)
-	)
-	(wire
-		(pts
 			(xy 96.52 106.68) (xy 96.52 104.14)
 		)
@@
 	(wire
 		(pts
+			(xy 114.3 49.53) (xy 114.3 63.5)
+		)
+		(stroke
+			(width 0)
+			(type default)
+		)
+	)
+	(wire
+		(pts
 			(xy 46.99 35.56) (xy 39.37 35.56)
 		)
@@
 	(wire
 		(pts
-			(xy 134.62 58.42) (xy 134.62 63.5)
-		)
-		(stroke
-			(width 0)
-			(type default)
-		)
-	)
-	(wire
-		(pts
-			(xy 137.16 58.42) (xy 137.16 63.5)
+			(xy 116.84 49.53) (xy 116.84 63.5)
 		)
 		(stroke
@@
 		)
 	)
-	(label "TCK"
-		(at 134.62 58.42 90)
-		(effects
-			(font
-				(size 1.27 1.27)
-			)
-			(justify left bottom)
-		)
-	)
 	(label "RXD0"
 		(at 93.98 93.98 180)
@@
 		)
 	)
-	(label "TDO"
-		(at 132.08 58.42 90)
-		(effects
-			(font
-				(size 1.27 1.27)
-			)
-			(justify left bottom)
-		)
-	)
 	(label "IO0"
 		(at 127 58.42 90)
@@
 		)
 	)
-	(label "TMS"
-		(at 139.7 58.42 90)
-		(effects
-			(font
-				(size 1.27 1.27)
-			)
-			(justify left bottom)
-		)
-	)
 	(label "IO0"
 		(at 46.99 43.18 0)
@@
 		)
 	)
+	(label "V3S-ESP32_RX"
+		(at 114.3 49.53 90)
+		(effects
+			(font
+				(size 1.27 1.27)
+			)
+			(justify left bottom)
+		)
+	)
 	(label "IO18"
 		(at 46.99 38.1 0)
@@
 		)
 	)
-	(label "TDI"
-		(at 137.16 58.42 90)
-		(effects
-			(font
+	(label "V3S-ESP32_TX"
+		(at 116.84 49.53 90)
+		(effects
+			(font
