File: MainBoard/MainBoard.kicad_pcb (KiCad board)
At the start: 2 copper layers, 55 x 90 mm, 163 parts, among them CN3 PJ-342, J1 1769, Q3 MMBT2222ALT1G, SW1 TS3735A 250GF 030, SW2 TS3735A 250GF 030, SW3 TS3735A 250GF 030, SW4 TS3735A 250GF 030, SW5 TS3735A 250GF 030, U1 V3S, U10 F35SQA512M-WWT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

Commit message: before moving esp32
Parts:
- moved J1 4.37 mm to (172.7, 117.7), turned to -90 degrees

Commit message: rotated ESP32
Parts:
- moved C31 6.85 mm to (126.8, 76.5), turned to 0 degrees
- moved C30 4.22 mm to (124.8, 76.5), turned to 180 degrees
- moved JP2 0.25 mm to (132.8, 92.8)
- turned U2 to 90 degrees
Routing:
- net I2S_SCK: track 32.6 -> 48.5 mm
- net I2S_PCMOUT: track 39.1 -> 54.2 mm
- net I2S_MCLK: track 30.3 -> 44.9 mm, vias 0 -> 2
- net /WiFi+BT/IO33: track 54.7 -> 42.5 mm
- net /WiFi+BT/TXD0: track 22.6 -> 10.6 mm
- net /WiFi+BT/RXD0: track 25.4 -> 13.5 mm
- net /WiFi+BT/IO32: track 20.3 -> 10.6 mm
- net +3.3V: track 461.7 -> 469.7 mm
- net I2S_WS: track 37.8 -> 45.0 mm
- net /WiFi+BT/IO25: track 31.9 -> 25.4 mm
- net /WiFi+BT/IO35: track 55.5 -> 49.1 mm
- net V3S-ESP32_RX: track 29.3 -> 24.7 mm
- net /WiFi+BT/IO34: track 37.0 -> 41.4 mm
- net V3S-ESP32_TX: track 29.6 -> 26.6 mm
- net PCM_CS: track 35.6 -> 34.0 mm
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